File: v3/pcb/v3.kicad_pcb (KiCad board)
At the start: 2 copper layers, 193 parts, among them SW1 SW_Push, SW10 SW_Push, SW11 SW_Push, SW12 SW_Push, SW13 SW_Push, SW14 SW_Push, SW15 SW_Push, SW16 SW_Push, SW17 SW_Push, SW18 SW_Push, SW19 SW_Push, SW2 SW_Push, SW20 SW_Push, SW21 SW_Push, SW22 SW_Push, SW23 SW_Push, SW24 SW_Push, SW25 SW_Push, SW26 SW_Push, SW27 SW_Push, SW28 SW_Push, SW29 SW_Push, SW3 SW_Push, SW30 SW_Push, SW31 SW_Push, SW32 SW_Push, SW33 SW_Push, SW34 SW_Push, SW35 SW_Push, SW36 SW_Push, SW37 SW_Push, SW38 SW_Push, SW39 SW_Push, SW4 SW_Push, SW40 SW_Push, SW41 SW_Push, SW42 SW_Push, SW43 SW_Push, SW44 SW_Push, SW45 SW_Push, SW46 SW_Push, SW47 SW_Push, SW48 SW_Push, SW49 SW_Push, SW5 SW_Push, SW50 SW_Push, SW51 SW_Push, SW52 SW_Push, SW53 SW_Push, SW54 SW_Push, SW55 SW_Push, SW56 SW_Push, SW57 SW_Push, SW58 SW_Push, SW59 SW_Push, SW6 SW_Push, SW60 SW_Push, SW61 SW_Push, SW62 SW_Push, SW63 SW_Push, SW64 SW_Push, SW65 SW_Push, SW66 SW_Push, SW67 SW_Push, SW68 SW_Push, SW69 SW_Push, SW7 SW_Push, SW70 SW_Push, SW71 SW_Push, SW72 SW_Push, SW73 SW_Push, SW74 SW_Push, SW75 SW_Push, SW76 SW_Push, SW77 SW_Push, SW78 SW_Push, SW79 SW_Push, SW8 SW_Push, SW80 SW_Push, SW81 SW_Push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

Commit message: Add new layout for v3
Parts:
- added D97: D, Diode_SMD:D_SOD-323F, B.Cu at (330.1, 142.3)
- added D98: D, Diode_SMD:D_SOD-323F, B.Cu at (363.5, 142.3)
- added D99: D, Diode_SMD:D_SOD-323F, B.Cu at (392.0, 142.3)
- added SW97: SW_Push, Switch_Keyboard_Cherry_MX:SW_Cherry_MX_PCB_1.00u, F.Cu at (325.0, 139.3)
- added SW98: SW_Push, Switch_Keyboard_Cherry_MX:SW_Cherry_MX_PCB_1.00u, F.Cu at (358.4, 139.3)
- added SW99: SW_Push, Switch_Keyboard_Cherry_MX:SW_Cherry_MX_PCB_1.00u, F.Cu at (386.9, 139.3)
- moved D86 369.2 mm to (411.1, 132.8)
- moved SW86 369.2 mm to (406.0, 129.8)
- moved U1 273.2 mm to (81.5, -14.5)
- moved D90 111.9 mm to (120.6, 142.3)
- moved SW90 111.9 mm to (115.5, 139.3)
- moved D91 97.6 mm to (158.7, 142.3)
- moved SW91 97.6 mm to (153.6, 139.3)
- moved D96 88.1 mm to (303.9, 142.3)
- moved SW96 88.1 mm to (298.8, 139.3)
- moved D95 83.3 mm to (280.1, 142.3)
- moved SW92 83.3 mm to (191.7, 139.3)
- moved SW95 83.3 mm to (275.0, 139.3)
- moved D92 83.3 mm to (196.8, 142.3)
- moved D94 73.8 mm to (256.3, 142.3)
- moved SW94 73.8 mm to (251.2, 139.3)
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Connections:
- D86 pad 1: ROW5 -> ROW4
- SW80 pad 1: COL13 -> COL12
- SW81 pad 1: COL14 -> COL13
- SW82 pad 1: COL15 -> COL14
- SW83 pad 1: COL16 -> COL15
- SW84 pad 1: COL17 -> COL16
- SW85 pad 1: COL18 -> COL17
- SW86 pad 1: COL0 -> COL18
- SW87 pad 1: COL1 -> COL0
- SW88 pad 1: COL2 -> COL1
- SW89 pad 1: COL6 -> COL2
- SW90 pad 1: COL10 -> COL4
- SW91 pad 1: COL11 -> COL6
- SW92 pad 1: COL12 -> COL8
- SW93 pad 1: COL13 -> COL10
- SW94 pad 1: COL14 -> COL11
- SW95 pad 1: COL15 -> COL12
- SW96 pad 1: COL17 -> COL13
Routing:
- net COL0: track 425.9 -> 108.9 mm
- net COL1: track 399.7 -> 85.1 mm
- net COL2: track 397.2 -> 112.8 mm
- net COL3: track 358.8 -> 90.8 mm
- net COL5: track 326.1 -> 90.8 mm
- net COL4: track 342.5 -> 109.9 mm
- net COL6: track 324.2 -> 113.8 mm
- net COL7: track 287.8 -> 94.8 mm
- net COL9: track 255.1 -> 94.8 mm
- net COL8: track 271.5 -> 113.8 mm
- net COL10: track 253.2 -> 119.7 mm
- net COL11: track 236.8 -> 118.8 mm
- net COL12: track 214.4 -> 112.8 mm
- net COL13: track 187.6 -> 112.8 mm
- net COL14: track 125.2 -> 76.2 mm
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
Commit message: Replace switch footprints with hotswap sockets
Parts:
- SW1, SW10, SW11, SW12, SW13, SW14, SW15, SW16, SW17, SW18, SW19, SW2, SW20, SW21, SW22, SW23, SW24, SW25, SW26, SW27, SW28, SW29, SW3, SW30, SW31, SW32, SW33, SW34, SW35, SW36, SW37, SW38, SW39, SW4, SW40, SW41, SW42, SW43, SW44, SW45, SW46, SW47, SW48, SW49, SW5, SW50, SW51, SW52, SW53, SW54, SW55, SW56, SW57, SW58, SW59, SW6, SW60, SW61, SW62, SW63, SW64, SW65, SW66, SW67, SW68, SW69, SW7, SW70, SW71, SW72, SW73, SW74, SW75, SW76, SW77, SW78, SW79, SW8, SW80, SW81, SW82, SW83, SW84, SW85, SW86, SW87, SW88, SW89, SW9, SW90, SW91, SW92, SW93, SW94, SW95, SW96, SW97, SW98, SW99: footprint Switch_Keyboard_Cherry_MX:SW_Cherry_MX_PCB_1.00u -> prettylib:MX_KAILH_SOCKET_1U
- U1: moved to B.Cu
- moved U1 273.6 mm to (350.5, 35.6)
Routing:
- net ROW1: track 371.5 -> 0.00 mm
- net ROW5: track 350.0 -> 0.00 mm
- net ROW2: track 347.7 -> 0.00 mm
- net ROW3: track 345.3 -> 0.00 mm
- net ROW4: track 340.5 -> 0.00 mm
- net ROW0: track 266.7 -> 0.00 mm
- net COL15: track 80.1 -> 0.00 mm
- net COL17: track 76.2 -> 0.00 mm
- net COL14: track 76.2 -> 0.00 mm
- net COL18: track 66.7 -> 0.00 mm
- net COL16: track 57.1 -> 0.00 mm
- net COL13: track 112.8 -> 93.8 mm
- net Net-(D9-Pad2): track 16.1 -> 0.00 mm
- net Net-(D6-Pad2): track 16.1 -> 0.00 mm
- net Net-(D13-Pad2): track 16.1 -> 0.00 mm
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
Commit message: Add level shifter and everything else for the RGBs
Parts:
- added C1: 100n, prettylib:SMD-0603, B.Cu at (39.6, 42.3)
- added C10: 100n, prettylib:SMD-0603, B.Cu at (249.2, 42.3)
- added C11: 100n, prettylib:SMD-0603, B.Cu at (268.2, 42.3)
- added C12: 100n, prettylib:SMD-0603, B.Cu at (287.3, 42.3)
- added C13: 100n, prettylib:SMD-0603, B.Cu at (306.3, 42.3)
- added C14: 100n, prettylib:SMD-0603, B.Cu at (39.6, 66.1)
- added C15: 100n, prettylib:SMD-0603, B.Cu at (58.7, 66.1)
- added C16: 100n, prettylib:SMD-0603, B.Cu at (77.7, 66.1)
- added C17: 100n, prettylib:SMD-0603, B.Cu at (96.8, 66.1)
- added C18: 100n, prettylib:SMD-0603, B.Cu at (115.8, 66.1)
- added C19: 100n, prettylib:SMD-0603, B.Cu at (134.9, 66.1)
- added C2: 100n, prettylib:SMD-0603, B.Cu at (77.7, 42.3)
- added C20: 100n, prettylib:SMD-0603, B.Cu at (153.9, 66.1)
- added C21: 100n, prettylib:SMD-0603, B.Cu at (173.0, 66.1)
- added C22: 100n, prettylib:SMD-0603, B.Cu at (192.0, 66.1)
- added C23: 100n, prettylib:SMD-0603, B.Cu at (211.1, 66.1)
- added C24: 100n, prettylib:SMD-0603, B.Cu at (230.1, 66.1)
- added C25: 100n, prettylib:SMD-0603, B.Cu at (249.2, 66.1)
- added C26: 100n, prettylib:SMD-0603, B.Cu at (268.2, 66.1)
- added C27: 100n, prettylib:SMD-0603, B.Cu at (296.8, 66.1)
- added C28: 100n, prettylib:SMD-0603, B.Cu at (330.1, 66.1)
- added C29: 100n, prettylib:SMD-0603, B.Cu at (353.9, 66.1)
- added C3: 100n, prettylib:SMD-0603, B.Cu at (96.8, 42.3)
- added C30: 100n, prettylib:SMD-0603, B.Cu at (373.0, 66.1)
- added C31: 100n, prettylib:SMD-0603, B.Cu at (392.0, 66.1)
- added C32: 100n, prettylib:SMD-0603, B.Cu at (411.1, 66.1)
- added C33: 100n, prettylib:SMD-0603, B.Cu at (44.4, 85.2)
- added C34: 100n, prettylib:SMD-0603, B.Cu at (68.2, 85.2)
- added C35: 100n, prettylib:SMD-0603, B.Cu at (87.2, 85.2)
- added C36: 100n, prettylib:SMD-0603, B.Cu at (106.3, 85.2)
- added C37: 100n, prettylib:SMD-0603, B.Cu at (125.3, 85.2)
- added C38: 100n, prettylib:SMD-0603, B.Cu at (144.4, 85.2)
- added C39: 100n, prettylib:SMD-0603, B.Cu at (163.4, 85.2)
- added C4: 100n, prettylib:SMD-0603, B.Cu at (115.8, 42.3)
- added C40: 100n, prettylib:SMD-0603, B.Cu at (182.5, 85.2)
- added C41: 100n, prettylib:SMD-0603, B.Cu at (201.5, 85.2)
- added C42: 100n, prettylib:SMD-0603, B.Cu at (220.6, 85.2)
- added C43: 100n, prettylib:SMD-0603, B.Cu at (239.6, 85.2)
- added C44: 100n, prettylib:SMD-0603, B.Cu at (258.7, 85.2)
- added C45: 100n, prettylib:SMD-0603, B.Cu at (277.7, 85.2)
- added C46: 100n, prettylib:SMD-0603, B.Cu at (301.5, 85.2)
- added C47: 100n, prettylib:SMD-0603, B.Cu at (330.1, 85.2)
- added C48: 100n, prettylib:SMD-0603, B.Cu at (353.9, 85.2)
- added C49: 100n, prettylib:SMD-0603, B.Cu at (373.0, 85.2)
- added C5: 100n, prettylib:SMD-0603, B.Cu at (134.9, 42.3)
- added C50: 100n, prettylib:SMD-0603, B.Cu at (392.0, 85.2)
- added C51: 100n, prettylib:SMD-0603, B.Cu at (411.1, 94.7)
- added C52: 100n, prettylib:SMD-0603, B.Cu at (46.7, 104.2)
- added C53: 100n, prettylib:SMD-0603, B.Cu at (72.9, 104.2)
- added C54: 100n, prettylib:SMD-0603, B.Cu at (92.0, 104.2)
- added C55: 100n, prettylib:SMD-0603, B.Cu at (111.0, 104.2)
- added C56: 100n, prettylib:SMD-0603, B.Cu at (130.1, 104.2)
- added C57: 100n, prettylib:SMD-0603, B.Cu at (149.1, 104.2)
- added C58: 100n, prettylib:SMD-0603, B.Cu at (168.2, 104.2)
- added C59: 100n, prettylib:SMD-0603, B.Cu at (187.2, 104.2)
- added C6: 100n, prettylib:SMD-0603, B.Cu at (163.4, 42.3)
- added C60: 100n, prettylib:SMD-0603, B.Cu at (206.3, 104.2)
- added C61: 100n, prettylib:SMD-0603, B.Cu at (225.3, 104.2)
- added C62: 100n, prettylib:SMD-0603, B.Cu at (244.4, 104.2)
- added C63: 100n, prettylib:SMD-0603, B.Cu at (263.4, 104.2)
- added C64: 100n, prettylib:SMD-0603, B.Cu at (294.4, 104.2)
- added C65: 100n, prettylib:SMD-0603, B.Cu at (330.1, 104.2)
- added C66: 100n, prettylib:SMD-0603, B.Cu at (353.9, 104.2)
- added C67: 100n, prettylib:SMD-0603, B.Cu at (373.0, 104.2)
- added C68: 100n, prettylib:SMD-0603, B.Cu at (392.0, 104.2)
- added C69: 100n, prettylib:SMD-0603, B.Cu at (51.5, 123.3)
- added C7: 100n, prettylib:SMD-0603, B.Cu at (182.5, 42.3)
- added C70: 100n, prettylib:SMD-0603, B.Cu at (82.5, 123.3)
- added C71: 100n, prettylib:SMD-0603, B.Cu at (101.5, 123.3)
- added C72: 100n, prettylib:SMD-0603, B.Cu at (120.6, 123.3)
- added C73: 100n, prettylib:SMD-0603, B.Cu at (139.6, 123.3)
- added C74: 100n, prettylib:SMD-0603, B.Cu at (158.7, 123.3)
- added C75: 100n, prettylib:SMD-0603, B.Cu at (177.7, 123.3)
- added C76: 100n, prettylib:SMD-0603, B.Cu at (196.8, 123.3)
- added C77: 100n, prettylib:SMD-0603, B.Cu at (215.8, 123.3)
- added C78: 100n, prettylib:SMD-0603, B.Cu at (234.9, 123.3)
- added C79: 100n, prettylib:SMD-0603, B.Cu at (253.9, 123.3)
- added C8: 100n, prettylib:SMD-0603, B.Cu at (201.5, 42.3)
- added C80: 100n, prettylib:SMD-0603, B.Cu at (280.1, 123.3)
- added C81: 100n, prettylib:SMD-0603, B.Cu at (303.9, 123.3)
- added C82: 100n, prettylib:SMD-0603, B.Cu at (330.1, 123.3)
- added C83: 100n, prettylib:SMD-0603, B.Cu at (353.9, 123.3)
- added C84: 100n, prettylib:SMD-0603, B.Cu at (373.0, 123.3)
- added C85: 100n, prettylib:SMD-0603, B.Cu at (392.0, 123.3)
- added C86: 100n, prettylib:SMD-0603, B.Cu at (411.1, 132.8)
- added C87: 100n, prettylib:SMD-0603, B.Cu at (42.0, 142.3)
- added C88: 100n, prettylib:SMD-0603, B.Cu at (65.8, 142.3)
- added C89: 100n, prettylib:SMD-0603, B.Cu at (89.6, 142.3)
- added C9: 100n, prettylib:SMD-0603, B.Cu at (220.6, 42.3)
- added C90: 100n, prettylib:SMD-0603, B.Cu at (113.4, 142.3)
- added C91: 100n, prettylib:SMD-0603, B.Cu at (151.5, 142.3)
- added C92: 100n, prettylib:SMD-0603, B.Cu at (196.8, 142.3)
- added C93: 100n, prettylib:SMD-0603, B.Cu at (230.1, 142.3)
- added C94: 100n, prettylib:SMD-0603, B.Cu at (256.3, 142.3)
- added C95: 100n, prettylib:SMD-0603, B.Cu at (280.1, 142.3)
- added C96: 100n, prettylib:SMD-0603, B.Cu at (303.9, 142.3)
- added C97: 100n, prettylib:SMD-0603, B.Cu at (330.1, 142.3)
- added C98: 100n, prettylib:SMD-0603, B.Cu at (363.5, 142.3)
- added C99: 100n, prettylib:SMD-0603, B.Cu at (392.0, 142.3)
- added RGB1: SK6812Mini-e, prettylib:SK6812_mini_e_flipable, F.Cu at (34.5, 39.3)
- added RGB10: SK6812Mini-e, prettylib:SK6812_mini_e_flipable, F.Cu at (244.1, 39.3)
- added RGB11: SK6812Mini-e, prettylib:SK6812_mini_e_flipable, F.Cu at (263.1, 39.3)
- added RGB12: SK6812Mini-e, prettylib:SK6812_mini_e_flipable, F.Cu at (282.2, 39.3)
- added RGB13: SK6812Mini-e, prettylib:SK6812_mini_e_flipable, F.Cu at (301.2, 39.3)
- added RGB14: SK6812Mini-e, prettylib:SK6812_mini_e_flipable, F.Cu at (34.5, 63.1)
- added RGB15: SK6812Mini-e, prettylib:SK6812_mini_e_flipable, F.Cu at (53.6, 63.1)
- added RGB16: SK6812Mini-e, prettylib:SK6812_mini_e_flipable, F.Cu at (72.6, 63.1)
- added RGB17: SK6812Mini-e, prettylib:SK6812_mini_e_flipable, F.Cu at (91.7, 63.1)
- added RGB18: SK6812Mini-e, prettylib:SK6812_mini_e_flipable, F.Cu at (110.7, 63.1)
- added RGB19: SK6812Mini-e, prettylib:SK6812_mini_e_flipable, F.Cu at (129.8, 63.1)
- added RGB2: SK6812Mini-e, prettylib:SK6812_mini_e_flipable, F.Cu at (72.6, 39.3)
- added RGB20: SK6812Mini-e, prettylib:SK6812_mini_e_flipable, F.Cu at (148.8, 63.1)
- added RGB21: SK6812Mini-e, prettylib:SK6812_mini_e_flipable, F.Cu at (167.9, 63.1)
- added RGB22: SK6812Mini-e, prettylib:SK6812_mini_e_flipable, F.Cu at (186.9, 63.1)
- added RGB23: SK6812Mini-e, prettylib:SK6812_mini_e_flipable, F.Cu at (206.0, 63.1)
- added RGB24: SK6812Mini-e, prettylib:SK6812_mini_e_flipable, F.Cu at (225.0, 63.1)
- added RGB25: SK6812Mini-e, prettylib:SK6812_mini_e_flipable, F.Cu at (244.1, 63.1)
- added RGB26: SK6812Mini, prettylib:SK6812_mini_e_flipable, F.Cu at (263.1, 63.1)
- added RGB27: SK6812Mini-e, prettylib:SK6812_mini_e_flipable, F.Cu at (291.7, 63.1)
- added RGB28: SK6812Mini-e, prettylib:SK6812_mini_e_flipable, F.Cu at (325.0, 63.1)
- added RGB29: SK6812Mini, prettylib:SK6812_mini_e_flipable, F.Cu at (348.9, 63.1)
- added RGB3: SK6812Mini-e, prettylib:SK6812_mini_e_flipable, F.Cu at (91.7, 39.3)
- added RGB30: SK6812Mini-e, prettylib:SK6812_mini_e_flipable, F.Cu at (367.9, 63.1)
- added RGB31: SK6812Mini-e, prettylib:SK6812_mini_e_flipable, F.Cu at (386.9, 63.1)
- added RGB32: SK6812Mini-e, prettylib:SK6812_mini_e_flipable, F.Cu at (406.0, 63.1)
- added RGB33: SK6812Mini-e, prettylib:SK6812_mini_e_flipable, F.Cu at (39.3, 82.2)
- added RGB34: SK6812Mini-e, prettylib:SK6812_mini_e_flipable, F.Cu at (63.1, 82.2)
- added RGB35: SK6812Mini-e, prettylib:SK6812_mini_e_flipable, F.Cu at (82.2, 82.2)
- added RGB36: SK6812Mini-e, prettylib:SK6812_mini_e_flipable, F.Cu at (101.2, 82.2)
- added RGB37: SK6812Mini-e, prettylib:SK6812_mini_e_flipable, F.Cu at (120.2, 82.2)
- added RGB38: SK6812Mini-e, prettylib:SK6812_mini_e_flipable, F.Cu at (139.3, 82.2)
- added RGB39: SK6812Mini-e, prettylib:SK6812_mini_e_flipable, F.Cu at (158.3, 82.2)
- added RGB4: SK6812Mini-e, prettylib:SK6812_mini_e_flipable, F.Cu at (110.7, 39.3)
- added RGB40: SK6812Mini-e, prettylib:SK6812_mini_e_flipable, F.Cu at (177.4, 82.2)
- added RGB41: SK6812Mini-e, prettylib:SK6812_mini_e_flipable, F.Cu at (196.4, 82.2)
- added RGB42: SK6812Mini-e, prettylib:SK6812_mini_e_flipable, F.Cu at (215.5, 82.2)
- added RGB43: SK6812Mini-e, prettylib:SK6812_mini_e_flipable, F.Cu at (234.6, 82.2)
- added RGB44: SK6812Mini-e, prettylib:SK6812_mini_e_flipable, F.Cu at (253.6, 82.2)
- added RGB45: SK6812Mini-e, prettylib:SK6812_mini_e_flipable, F.Cu at (272.6, 82.2)
- added RGB46: SK6812Mini, prettylib:SK6812_mini_e_flipable, F.Cu at (296.5, 82.2)
- added RGB47: SK6812Mini-e, prettylib:SK6812_mini_e_flipable, F.Cu at (325.0, 82.2)
- added RGB48: SK6812Mini-e, prettylib:SK6812_mini_e_flipable, F.Cu at (348.9, 82.2)
- added RGB49: SK6812Mini, prettylib:SK6812_mini_e_flipable, F.Cu at (367.9, 82.2)
- added RGB5: SK6812Mini-e, prettylib:SK6812_mini_e_flipable, F.Cu at (129.8, 39.3)
- added RGB50: SK6812Mini-e, prettylib:SK6812_mini_e_flipable, F.Cu at (386.9, 82.2)
- added RGB51: SK6812Mini-e, prettylib:SK6812_mini_e_flipable, F.Cu at (406.0, 91.7)
- added RGB52: SK6812Mini-e, prettylib:SK6812_mini_e_flipable, F.Cu at (41.7, 101.2)
- added RGB53: SK6812Mini-e, prettylib:SK6812_mini_e_flipable, F.Cu at (67.9, 101.2)
- added RGB54: SK6812Mini-e, prettylib:SK6812_mini_e_flipable, F.Cu at (86.9, 101.2)
- added RGB55: SK6812Mini-e, prettylib:SK6812_mini_e_flipable, F.Cu at (106.0, 101.2)
- added RGB56: SK6812Mini-e, prettylib:SK6812_mini_e_flipable, F.Cu at (125.0, 101.2)
- added RGB57: SK6812Mini-e, prettylib:SK6812_mini_e_flipable, F.Cu at (144.1, 101.2)
- added RGB58: SK6812Mini-e, prettylib:SK6812_mini_e_flipable, F.Cu at (163.1, 101.2)
- added RGB59: SK6812Mini-e, prettylib:SK6812_mini_e_flipable, F.Cu at (182.2, 101.2)
- added RGB6: SK6812Mini, prettylib:SK6812_mini_e_flipable, F.Cu at (158.3, 39.3)
- added RGB60: SK6812Mini-e, prettylib:SK6812_mini_e_flipable, F.Cu at (201.2, 101.2)
- added RGB61: SK6812Mini-e, prettylib:SK6812_mini_e_flipable, F.Cu at (220.3, 101.2)
- added RGB62: SK6812Mini-e, prettylib:SK6812_mini_e_flipable, F.Cu at (239.3, 101.2)
- added RGB63: SK6812Mini-e, prettylib:SK6812_mini_e_flipable, F.Cu at (258.4, 101.2)
- added RGB64: SK6812Mini-e, prettylib:SK6812_mini_e_flipable, F.Cu at (289.3, 101.2)
- added RGB65: SK6812Mini-e, prettylib:SK6812_mini_e_flipable, F.Cu at (325.0, 101.2)
- added RGB66: SK6812Mini, prettylib:SK6812_mini_e_flipable, F.Cu at (348.9, 101.2)
- added RGB67: SK6812Mini-e, prettylib:SK6812_mini_e_flipable, F.Cu at (367.9, 101.2)
- added RGB68: SK6812Mini-e, prettylib:SK6812_mini_e_flipable, F.Cu at (386.9, 101.2)
- added RGB69: SK6812Mini, prettylib:SK6812_mini_e_flipable, F.Cu at (46.4, 120.2)
- added RGB7: SK6812Mini-e, prettylib:SK6812_mini_e_flipable, F.Cu at (177.4, 39.3)
- added RGB70: SK6812Mini-e, prettylib:SK6812_mini_e_flipable, F.Cu at (77.4, 120.2)
- added RGB71: SK6812Mini-e, prettylib:SK6812_mini_e_flipable, F.Cu at (96.4, 120.2)
- added RGB72: SK6812Mini-e, prettylib:SK6812_mini_e_flipable, F.Cu at (115.5, 120.2)
- added RGB73: SK6812Mini-e, prettylib:SK6812_mini_e_flipable, F.Cu at (134.5, 120.2)
- added RGB74: SK6812Mini-e, prettylib:SK6812_mini_e_flipable, F.Cu at (153.6, 120.2)
- added RGB75: SK6812Mini-e, prettylib:SK6812_mini_e_flipable, F.Cu at (172.6, 120.2)
- added RGB76: SK6812Mini-e, prettylib:SK6812_mini_e_flipable, F.Cu at (191.7, 120.2)
- added RGB77: SK6812Mini-e, prettylib:SK6812_mini_e_flipable, F.Cu at (210.7, 120.2)
- added RGB78: SK6812Mini-e, prettylib:SK6812_mini_e_flipable, F.Cu at (229.8, 120.2)
- added RGB79: SK6812Mini-e, prettylib:SK6812_mini_e_flipable, F.Cu at (248.8, 120.2)
- added RGB8: SK6812Mini-e, prettylib:SK6812_mini_e_flipable, F.Cu at (196.4, 39.3)
- added RGB80: SK6812Mini-e, prettylib:SK6812_mini_e_flipable, F.Cu at (275.0, 120.2)
- added RGB81: SK6812Mini-e, prettylib:SK6812_mini_e_flipable, F.Cu at (298.8, 120.2)
- added RGB82: SK6812Mini-e, prettylib:SK6812_mini_e_flipable, F.Cu at (325.0, 120.2)
- added RGB83: SK6812Mini-e, prettylib:SK6812_mini_e_flipable, F.Cu at (348.9, 120.2)
- added RGB84: SK6812Mini-e, prettylib:SK6812_mini_e_flipable, F.Cu at (367.9, 120.2)
- added RGB85: SK6812Mini-e, prettylib:SK6812_mini_e_flipable, F.Cu at (386.9, 120.2)
- added RGB86: SK6812Mini, prettylib:SK6812_mini_e_flipable, F.Cu at (406.0, 129.8)
- added RGB87: SK6812Mini-e, prettylib:SK6812_mini_e_flipable, F.Cu at (36.9, 139.3)
- added RGB88: SK6812Mini-e, prettylib:SK6812_mini_e_flipable, F.Cu at (60.7, 139.3)
- added RGB89: SK6812Mini, prettylib:SK6812_mini_e_flipable, F.Cu at (84.5, 139.3)
- added RGB9: SK6812Mini, prettylib:SK6812_mini_e_flipable, F.Cu at (215.5, 39.3)
- added RGB90: SK6812Mini-e, prettylib:SK6812_mini_e_flipable, F.Cu at (108.3, 139.3)
- added RGB91: SK6812Mini-e, prettylib:SK6812_mini_e_flipable, F.Cu at (146.4, 139.3)
- added RGB92: SK6812Mini-e, prettylib:SK6812_mini_e_flipable, F.Cu at (191.7, 139.3)
- added RGB93: SK6812Mini-e, prettylib:SK6812_mini_e_flipable, F.Cu at (225.0, 139.3)
- added RGB94: SK6812Mini-e, prettylib:SK6812_mini_e_flipable, F.Cu at (251.2, 139.3)
- added RGB95: SK6812Mini-e, prettylib:SK6812_mini_e_flipable, F.Cu at (275.0, 139.3)
- added RGB96: SK6812Mini-e, prettylib:SK6812_mini_e_flipable, F.Cu at (298.8, 139.3)
- added RGB97: SK6812Mini-e, prettylib:SK6812_mini_e_flipable, F.Cu at (325.0, 139.3)
- added RGB98: SK6812Mini-e, prettylib:SK6812_mini_e_flipable, F.Cu at (358.4, 139.3)
- added RGB99: SK6812Mini-e, prettylib:SK6812_mini_e_flipable, F.Cu at (386.9, 139.3)
- added TP1: Joystick X, TestPoint:TestPoint_THTPad_D1.5mm_Drill0.7mm, F.Cu at (617.2, 40.6)
- added TP2: Joystick VDD, TestPoint:TestPoint_THTPad_D1.5mm_Drill0.7mm, F.Cu at (609.6, 53.3)
- added TP3: Joystick Y, TestPoint:TestPoint_THTPad_D1.5mm_Drill0.7mm, F.Cu at (594.4, 78.7)
- added TP4: Joystick GND, TestPoint:TestPoint_THTPad_D1.5mm_Drill0.7mm, F.Cu at (614.7, 25.4)
- added U2: SN74LVC1T45DCK, Package_TO_SOT_SMD:SOT-363_SC-70-6, F.Cu at (539.1, 38.9)
- moved U1 138.6 mm to (356.6, 174.1), turned to 180 degrees
- moved SW51 136.1 mm to (412.1, 227.6)
- moved SW52 136.1 mm to (47.8, 237.2)
- moved SW53 136.1 mm to (74.0, 237.2)
- moved SW54 136.1 mm to (93.0, 237.2)
- moved SW55 136.1 mm to (112.1, 237.2)
- moved SW56 136.1 mm to (131.1, 237.2)
- moved SW57 136.1 mm to (150.2, 237.2)
- moved SW59 136.1 mm to (188.3, 237.2)
- moved SW61 136.1 mm to (226.4, 237.2)
- moved SW62 136.1 mm to (245.4, 237.2)
- moved SW63 136.1 mm to (264.5, 237.2)
- moved SW67 136.1 mm to (374.0, 237.2)
- moved SW68 136.1 mm to (393.1, 237.2)
- moved SW69 136.1 mm to (52.5, 256.2)
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Connections:
- D1 pad 1: ROW0 -> COL1
- D10 pad 1: ROW0 -> COL1
- D11 pad 1: ROW0 -> COL1
- D12 pad 1: ROW0 -> COL1
- D13 pad 1: ROW0 -> COL1
- D2 pad 1: ROW0 -> COL1
- D3 pad 1: ROW0 -> COL1
- D4 pad 1: ROW0 -> COL1
- D5 pad 1: ROW0 -> COL1
- D6 pad 1: ROW0 -> COL1
- D7 pad 1: ROW0 -> COL1
- D8 pad 1: ROW0 -> COL1
- D9 pad 1: ROW0 -> COL1
- SW15 pad 1: COL1 -> Net-(SW15-Pad1)
- SW34 pad 1: COL1 -> Net-(SW15-Pad1)
- SW53 pad 1: COL1 -> Net-(SW15-Pad1)
- SW88 pad 1: COL1 -> Net-(SW15-Pad1)
- U1 pad 1: unconnected-(U1-Pad1) -> GND
- U1 pad 10: COL8 -> COL16
- U1 pad 11: COL9 -> COL15
- U1 pad 12: COL10 -> COL14
- U1 pad 13: COL11 -> COL13
- U1 pad 15: unconnected-(U1-Pad15) -> 3V3REF
- U1 pad 16: COL13 -> COL11
- U1 pad 17: COL14 -> COL10
- U1 pad 18: COL15 -> COL9
- U1 pad 19: COL16 -> COL8
- U1 pad 2: COL0 -> ROW5
- U1 pad 20: COL17 -> COL7
- U1 pad 21: COL18 -> COL6
- U1 pad 22: ROW0 -> COL5
- U1 pad 23: ROW1 -> COL4
- U1 pad 24: ROW2 -> COL3
- U1 pad 3: COL1 -> ROW4
- U1 pad 30: ROW3 -> COL2
- U1 pad 31: ROW4 -> COL1
- U1 pad 32: ROW5 -> COL0
- U1 pad 33: unconnected-(U1-Pad33) -> JOYSTICK_X
- U1 pad 34: unconnected-(U1-Pad34) -> JOYSTICK_Y
- U1 pad 35: unconnected-(U1-Pad35) -> RGB_3V3_DATA
- U1 pad 4: COL2 -> ROW3
- U1 pad 5: COL3 -> ROW2
- U1 pad 54: unconnected-(U1-Pad54) -> VUSB
- U1 pad 6: COL4 -> ROW1
- U1 pad 7: COL5 -> COL1
- U1 pad 8: COL6 -> COL18
- U1 pad 9: COL7 -> COL17
Routing:
- net COL10: track 121.1 -> 0.00 mm
- net COL11: track 118.7 -> 0.00 mm
- net COL6: track 115.2 -> 0.00 mm
- net COL12: track 114.9 -> 0.00 mm
- net COL8: track 113.9 -> 0.00 mm
- net COL2: track 112.8 -> 0.00 mm
- net COL4: track 110.0 -> 0.00 mm
- net COL0: track 104.5 -> 0.00 mm
- net COL7: track 94.8 -> 0.00 mm
- net COL9: track 94.7 -> 0.00 mm
- net COL13: track 93.8 -> 0.00 mm
- net COL5: track 90.9 -> 0.00 mm
- net COL3: track 90.8 -> 0.00 mm
- net COL1: track 85.1 -> 0.00 mm
Other:
- board outline added: 3.4 x 4 mm

Commit message: Align LED:s and add stabilizer holes
Parts:
- added H1: MountingHole, MountingHole:MountingHole_3.5mm, F.Cu at (22.9, 17.8)
- added H2: MountingHole, MountingHole:MountingHole_3.5mm, F.Cu at (420.4, 17.8)
- added H3: MountingHole, MountingHole:MountingHole_3.5mm, F.Cu at (22.9, 147.3)
- added H4: MountingHole, MountingHole:MountingHole_3.5mm, F.Cu at (420.4, 147.5)
- added H5: MountingHole, MountingHole:MountingHole_3.5mm, F.Cu at (229.9, 19.1)
- added H6: MountingHole, MountingHole:MountingHole_3.5mm, F.Cu at (226.1, 148.6)
- SW27, SW64, SW69, SW91, SW92, SW98: footprint prettylib:MX_KAILH_SOCKET_1U -> zekeyboard:MX_KAILH_SOCKET_2U_STAB
- SW51, SW86: footprint prettylib:MX_KAILH_SOCKET_1U -> zekeyboard:MX_KAILH_SOCKET_2U_STAB_VERT
- moved U2 224.4 mm to (314.8, 45.4)
- moved TP1 208.8 mm to (408.9, 25.4)
- moved TP4 206.5 mm to (408.9, 43.2)
- moved TP2 202.0 mm to (408.9, 30.5)
- moved TP3 190.4 mm to (408.9, 35.6)
- moved SW69 141.1 mm to (46.5, 115.2)
- moved SW70 141.1 mm to (77.4, 115.2)
- moved SW71 141.1 mm to (96.5, 115.2)
- moved SW72 141.1 mm to (115.5, 115.2)
- moved SW73 141.1 mm to (134.6, 115.2)
- moved SW75 141.1 mm to (172.7, 115.2)
- moved SW76 141.1 mm to (191.7, 115.2)
- moved SW77 141.1 mm to (210.8, 115.2)
- moved SW78 141.1 mm to (229.8, 115.2)
- moved SW80 141.1 mm to (275.1, 115.2)
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Other:
- board size 3.4 x 4 mm -> 407.7 x 139.9 mm

Commit message: Reorient LEDs and started on USB
Parts:
- RGB26, RGB29, RGB46, RGB49, RGB6, RGB66, RGB69, RGB86, RGB89, RGB9: value SK6812Mini -> SK6812Mini-e
- SW69: footprint zekeyboard:MX_KAILH_SOCKET_2U_STAB -> prettylib:MX_KAILH_SOCKET_1U
- moved U2 6.03 mm to (314.0, 39.4)
Connections:
- RGB1 pad 4: RGB_DATA -> Net-(RGB2-Pad2)
- RGB10 pad 4: Net-(RGB10-Pad4) -> Net-(RGB11-Pad2)
- RGB11 pad 4: Net-(RGB10-Pad2) -> Net-(RGB12-Pad2)
- RGB12 pad 4: Net-(RGB11-Pad2) -> Net-(RGB13-Pad2)
- RGB13 pad 4: Net-(RGB12-Pad2) -> RGB_DATA
- RGB14 pad 3: GND -> Net-(RGB14-Pad3)
- RGB14 pad 4: Net-(RGB13-Pad2) -> Net-(RGB1-Pad2)
- RGB15 pad 3: GND -> Net-(RGB14-Pad3)
- RGB16 pad 3: GND -> Net-(RGB14-Pad3)
- RGB17 pad 3: GND -> Net-(RGB14-Pad3)
- RGB18 pad 3: GND -> Net-(RGB14-Pad3)
- RGB19 pad 3: GND -> Net-(RGB14-Pad3)
- RGB2 pad 4: Net-(RGB1-Pad2) -> Net-(RGB3-Pad2)
- RGB20 pad 3: GND -> Net-(RGB14-Pad3)
- RGB21 pad 3: GND -> Net-(RGB14-Pad3)
- RGB22 pad 3: GND -> Net-(RGB14-Pad3)
- RGB23 pad 3: GND -> Net-(RGB14-Pad3)
- RGB24 pad 3: GND -> Net-(RGB14-Pad3)
- RGB25 pad 3: GND -> Net-(RGB14-Pad3)
- RGB26 pad 1: Net-(RGB26-Pad1) -> RGB_VDD
- RGB26 pad 2: GND -> Net-(RGB26-Pad2)
- RGB26 pad 3: Net-(RGB25-Pad2) -> Net-(RGB14-Pad3)
- RGB26 pad 4: RGB_VDD -> Net-(RGB25-Pad2)
- RGB27 pad 3: GND -> Net-(RGB14-Pad3)
- RGB27 pad 4: Net-(RGB26-Pad1) -> Net-(RGB26-Pad2)
- RGB28 pad 3: GND -> Net-(RGB14-Pad3)
- RGB29 pad 1: Net-(RGB29-Pad1) -> RGB_VDD
- RGB29 pad 2: GND -> Net-(RGB29-Pad2)
- RGB29 pad 3: Net-(RGB28-Pad2) -> Net-(RGB14-Pad3)
- RGB29 pad 4: RGB_VDD -> Net-(RGB28-Pad2)
- RGB3 pad 4: Net-(RGB2-Pad2) -> Net-(RGB4-Pad2)
- RGB30 pad 3: GND -> Net-(RGB14-Pad3)
- RGB30 pad 4: Net-(RGB29-Pad1) -> Net-(RGB29-Pad2)
- RGB31 pad 3: GND -> Net-(RGB14-Pad3)
- RGB32 pad 2: Net-(RGB32-Pad2) -> Net-(RGB51-Pad4)
- RGB32 pad 3: GND -> Net-(RGB14-Pad3)
- RGB33 pad 2: Net-(RGB33-Pad2) -> Net-(RGB52-Pad4)
- RGB33 pad 4: Net-(RGB32-Pad2) -> Net-(RGB33-Pad4)
- RGB34 pad 2: Net-(RGB34-Pad2) -> Net-(RGB33-Pad4)
- RGB34 pad 4: Net-(RGB33-Pad2) -> Net-(RGB34-Pad4)
- RGB35 pad 2: Net-(RGB35-Pad2) -> Net-(RGB34-Pad4)
- RGB35 pad 4: Net-(RGB34-Pad2) -> Net-(RGB35-Pad4)
- RGB36 pad 2: Net-(RGB36-Pad2) -> Net-(RGB35-Pad4)
- RGB36 pad 4: Net-(RGB35-Pad2) -> Net-(RGB36-Pad4)
- RGB37 pad 2: Net-(RGB37-Pad2) -> Net-(RGB36-Pad4)
- RGB37 pad 4: Net-(RGB36-Pad2) -> Net-(RGB37-Pad4)
- RGB38 pad 2: Net-(RGB38-Pad2) -> Net-(RGB37-Pad4)
- RGB38 pad 4: Net-(RGB37-Pad2) -> Net-(RGB38-Pad4)
- RGB39 pad 2: Net-(RGB39-Pad2) -> Net-(RGB38-Pad4)
- RGB39 pad 4: Net-(RGB38-Pad2) -> Net-(RGB39-Pad4)
- RGB4 pad 4: Net-(RGB3-Pad2) -> Net-(RGB4-Pad4)
- RGB40 pad 2: Net-(RGB40-Pad2) -> Net-(RGB39-Pad4)
- RGB40 pad 4: Net-(RGB39-Pad2) -> Net-(RGB40-Pad4)
- RGB41 pad 2: Net-(RGB41-Pad2) -> Net-(RGB40-Pad4)
- RGB41 pad 4: Net-(RGB40-Pad2) -> Net-(RGB41-Pad4)
- RGB42 pad 2: Net-(RGB42-Pad2) -> Net-(RGB41-Pad4)
- RGB42 pad 4: Net-(RGB41-Pad2) -> Net-(RGB42-Pad4)
- RGB43 pad 2: Net-(RGB43-Pad2) -> Net-(RGB42-Pad4)
- RGB43 pad 4: Net-(RGB42-Pad2) -> Net-(RGB44-Pad2)
- RGB44 pad 4: Net-(RGB43-Pad2) -> Net-(RGB45-Pad2)
- RGB45 pad 4: Net-(RGB44-Pad2) -> Net-(RGB46-Pad2)
- RGB46 pad 1: Net-(RGB46-Pad1) -> RGB_VDD
- RGB46 pad 2: GND -> Net-(RGB46-Pad2)
- RGB46 pad 3: Net-(RGB45-Pad2) -> GND
- RGB46 pad 4: RGB_VDD -> Net-(RGB47-Pad2)
- RGB47 pad 4: Net-(RGB46-Pad1) -> Net-(RGB48-Pad2)
- RGB48 pad 4: Net-(RGB47-Pad2) -> Net-(RGB49-Pad2)
- RGB49 pad 1: Net-(RGB49-Pad1) -> RGB_VDD
- RGB49 pad 2: GND -> Net-(RGB49-Pad2)
- RGB49 pad 3: Net-(RGB48-Pad2) -> GND
- RGB49 pad 4: RGB_VDD -> Net-(RGB50-Pad2)
- RGB5 pad 2: Net-(RGB5-Pad2) -> Net-(RGB4-Pad4)
- RGB5 pad 4: Net-(RGB4-Pad2) -> Net-(RGB6-Pad2)
- RGB50 pad 4: Net-(RGB49-Pad1) -> Net-(RGB51-Pad2)
- RGB51 pad 4: Net-(RGB50-Pad2) -> Net-(RGB51-Pad4)
- RGB52 pad 4: Net-(RGB51-Pad2) -> Net-(RGB52-Pad4)
- RGB6 pad 1: Net-(RGB6-Pad1) -> RGB_VDD
- RGB6 pad 2: GND -> Net-(RGB6-Pad2)
- RGB6 pad 3: Net-(RGB5-Pad2) -> GND
- RGB6 pad 4: RGB_VDD -> Net-(RGB7-Pad2)
- RGB66 pad 1: Net-(RGB66-Pad1) -> RGB_VDD
- RGB66 pad 2: GND -> Net-(RGB66-Pad2)
- RGB66 pad 3: Net-(RGB65-Pad2) -> GND
- RGB66 pad 4: RGB_VDD -> Net-(RGB65-Pad2)
- RGB67 pad 4: Net-(RGB66-Pad1) -> Net-(RGB66-Pad2)
- RGB69 pad 1: Net-(RGB69-Pad1) -> Net-(RGB86-Pad1)
- RGB69 pad 2: GND -> Net-(RGB87-Pad4)
- RGB69 pad 3: Net-(RGB68-Pad2) -> GND
- RGB69 pad 4: RGB_VDD -> Net-(RGB69-Pad4)
- RGB7 pad 4: Net-(RGB6-Pad1) -> Net-(RGB8-Pad2)
- RGB70 pad 1: RGB_VDD -> Net-(RGB86-Pad1)
- RGB70 pad 2: Net-(RGB70-Pad2) -> Net-(RGB69-Pad4)
- RGB70 pad 4: Net-(RGB69-Pad1) -> Net-(RGB70-Pad4)
- RGB71 pad 1: RGB_VDD -> Net-(RGB86-Pad1)
- RGB71 pad 2: Net-(RGB71-Pad2) -> Net-(RGB70-Pad4)
- RGB71 pad 4: Net-(RGB70-Pad2) -> Net-(RGB71-Pad4)
- RGB72 pad 1: RGB_VDD -> Net-(RGB86-Pad1)
- RGB72 pad 2: Net-(RGB72-Pad2) -> Net-(RGB71-Pad4)
- RGB72 pad 4: Net-(RGB71-Pad2) -> Net-(RGB72-Pad4)
- RGB73 pad 1: RGB_VDD -> Net-(RGB86-Pad1)
- RGB73 pad 2: Net-(RGB73-Pad2) -> Net-(RGB72-Pad4)
- RGB73 pad 4: Net-(RGB72-Pad2) -> Net-(RGB73-Pad4)
- RGB74 pad 1: RGB_VDD -> Net-(RGB86-Pad1)
- RGB74 pad 2: Net-(RGB74-Pad2) -> Net-(RGB73-Pad4)
- RGB74 pad 4: Net-(RGB73-Pad2) -> Net-(RGB75-Pad2)
- RGB75 pad 1: RGB_VDD -> Net-(RGB86-Pad1)
- RGB75 pad 4: Net-(RGB74-Pad2) -> Net-(RGB76-Pad2)
- RGB76 pad 1: RGB_VDD -> Net-(RGB86-Pad1)
- RGB76 pad 4: Net-(RGB75-Pad2) -> Net-(RGB77-Pad2)
- RGB77 pad 1: RGB_VDD -> Net-(RGB86-Pad1)
- RGB77 pad 4: Net-(RGB76-Pad2) -> Net-(RGB78-Pad2)
- RGB78 pad 1: RGB_VDD -> Net-(RGB86-Pad1)
- RGB78 pad 4: Net-(RGB77-Pad2) -> Net-(RGB79-Pad2)
- RGB79 pad 1: RGB_VDD -> Net-(RGB86-Pad1)
- RGB79 pad 4: Net-(RGB78-Pad2) -> Net-(RGB80-Pad2)
- RGB8 pad 4: Net-(RGB7-Pad2) -> Net-(RGB9-Pad2)
- RGB80 pad 1: RGB_VDD -> Net-(RGB86-Pad1)
- RGB80 pad 4: Net-(RGB79-Pad2) -> Net-(RGB81-Pad2)
- RGB81 pad 1: RGB_VDD -> Net-(RGB86-Pad1)
- RGB81 pad 4: Net-(RGB80-Pad2) -> Net-(RGB82-Pad2)
- RGB82 pad 1: RGB_VDD -> Net-(RGB86-Pad1)
- RGB82 pad 4: Net-(RGB81-Pad2) -> Net-(RGB83-Pad2)
- RGB83 pad 1: RGB_VDD -> Net-(RGB86-Pad1)
- RGB83 pad 4: Net-(RGB82-Pad2) -> Net-(RGB84-Pad2)
- RGB84 pad 1: RGB_VDD -> Net-(RGB86-Pad1)
- RGB84 pad 4: Net-(RGB83-Pad2) -> Net-(RGB85-Pad2)
- RGB85 pad 1: RGB_VDD -> Net-(RGB86-Pad1)
- RGB85 pad 4: Net-(RGB84-Pad2) -> Net-(RGB85-Pad4)
- RGB86 pad 2: GND -> Net-(RGB85-Pad4)
- RGB86 pad 3: Net-(RGB85-Pad2) -> GND
- RGB86 pad 4: RGB_VDD -> Net-(RGB68-Pad2)
- RGB87 pad 4: Net-(RGB86-Pad1) -> Net-(RGB87-Pad4)
- RGB89 pad 1: Net-(RGB89-Pad1) -> RGB_VDD
- RGB89 pad 2: GND -> Net-(RGB89-Pad2)
- RGB89 pad 3: Net-(RGB88-Pad2) -> GND
- RGB89 pad 4: RGB_VDD -> Net-(RGB88-Pad2)
- RGB9 pad 1: Net-(RGB10-Pad4) -> RGB_VDD
- RGB9 pad 2: GND -> Net-(RGB9-Pad2)
- RGB9 pad 3: Net-(RGB8-Pad2) -> GND
- RGB9 pad 4: RGB_VDD -> Net-(RGB10-Pad2)
- RGB90 pad 4: Net-(RGB89-Pad1) -> Net-(RGB89-Pad2)

Commit message: Finished USB and add pinouts for teensy
Parts:
- added F1: 3A, prettylib:Fuse_1206_3216Metric, F.Cu at (387.4, 24.1)
- added FB1: FerriteBead, Resistor_SMD:R_0402_1005Metric, F.Cu at (374.6, 21.6)
- added J1: USB_C_Receptacle_USB2.0, Connector_USB:USB_C_Receptacle_HRO_TYPE-C-31-M-12, F.Cu at (378.6, 12.5)
- added J2: Conn_01x21, Connector_PinHeader_2.00mm:PinHeader_1x21_P2.00mm_Vertical, F.Cu at (420.1, 28.1)
- added Q1: AO3401A, prettylib:SOT-23, F.Cu at (383.5, 27.9)
- added R1: 5.1k, Resistor_SMD:R_0603_1608Metric, F.Cu at (367.8, 22.0)
- added R2: 5.1k, Resistor_SMD:R_0603_1608Metric, F.Cu at (361.3, 22.0)
- added TP5: D+, TestPoint:TestPoint_THTPad_D1.5mm_Drill0.7mm, F.Cu at (396.0, 16.5)
- added TP6: D-, TestPoint:TestPoint_THTPad_D1.5mm_Drill0.7mm, F.Cu at (392.2, 16.5)
- added TP7: USB_VBUS, TestPoint:TestPoint_THTPad_D1.5mm_Drill0.7mm, F.Cu at (388.1, 16.5)
- added U3: LMV321, prettylib:SOT-23-5, F.Cu at (396.2, 22.9)
- added U4: SRV0504, prettylib:SOT-23-6, F.Cu at (389.9, 27.9)
- moved TP1 76.8 mm to (332.7, 15.7), turned to 180 degrees
- moved TP2 71.1 mm to (339.3, 15.7)
- moved TP3 66.5 mm to (345.4, 15.7), turned to 180 degrees
- moved TP4 63.2 mm to (352.0, 15.7)
- moved U1 1.21 mm to (350.5, 34.3)
Connections:
- C1 pad 1: RGB_VDD -> +5V
- C10 pad 1: RGB_VDD -> +5V
- C11 pad 1: RGB_VDD -> +5V
- C12 pad 1: RGB_VDD -> +5V
- C13 pad 1: RGB_VDD -> +5V
- C14 pad 1: RGB_VDD -> +5V
- C15 pad 1: RGB_VDD -> +5V
- C16 pad 1: RGB_VDD -> +5V
- C17 pad 1: RGB_VDD -> +5V
- C18 pad 1: RGB_VDD -> +5V
- C19 pad 1: RGB_VDD -> +5V
- C2 pad 1: RGB_VDD -> +5V
- C20 pad 1: RGB_VDD -> +5V
- C21 pad 1: RGB_VDD -> +5V
- C22 pad 1: RGB_VDD -> +5V
- C23 pad 1: RGB_VDD -> +5V
- C24 pad 1: RGB_VDD -> +5V
- C25 pad 1: RGB_VDD -> +5V
- C26 pad 1: RGB_VDD -> +5V
- C27 pad 1: RGB_VDD -> +5V
- C28 pad 1: RGB_VDD -> +5V
- C29 pad 1: RGB_VDD -> +5V
- C3 pad 1: RGB_VDD -> +5V
- C30 pad 1: RGB_VDD -> +5V
- C31 pad 1: RGB_VDD -> +5V
- C32 pad 1: RGB_VDD -> +5V
- C33 pad 1: RGB_VDD -> +5V
- C34 pad 1: RGB_VDD -> +5V
- C35 pad 1: RGB_VDD -> +5V
- C36 pad 1: RGB_VDD -> +5V
- C37 pad 1: RGB_VDD -> +5V
- C38 pad 1: RGB_VDD -> +5V
- C39 pad 1: RGB_VDD -> +5V
- C4 pad 1: RGB_VDD -> +5V
- C40 pad 1: RGB_VDD -> +5V
- C41 pad 1: RGB_VDD -> +5V
- C42 pad 1: RGB_VDD -> +5V
- C43 pad 1: RGB_VDD -> +5V
- C44 pad 1: RGB_VDD -> +5V
- C45 pad 1: RGB_VDD -> +5V
- C46 pad 1: RGB_VDD -> +5V
- C47 pad 1: RGB_VDD -> +5V
- C48 pad 1: RGB_VDD -> +5V
- C49 pad 1: RGB_VDD -> +5V
- C5 pad 1: RGB_VDD -> +5V
- C50 pad 1: RGB_VDD -> +5V
- C51 pad 1: RGB_VDD -> +5V
- C52 pad 1: RGB_VDD -> +5V
- C53 pad 1: RGB_VDD -> +5V
- C54 pad 1: RGB_VDD -> +5V
- C55 pad 1: RGB_VDD -> +5V
- C56 pad 1: RGB_VDD -> +5V
- C57 pad 1: RGB_VDD -> +5V
- C58 pad 1: RGB_VDD -> +5V
- C59 pad 1: RGB_VDD -> +5V
- C6 pad 1: RGB_VDD -> +5V
- C60 pad 1: RGB_VDD -> +5V
- C61 pad 1: RGB_VDD -> +5V
- C62 pad 1: RGB_VDD -> +5V
- C63 pad 1: RGB_VDD -> +5V
- C64 pad 1: RGB_VDD -> +5V
- C65 pad 1: RGB_VDD -> +5V
- C66 pad 1: RGB_VDD -> +5V
- C67 pad 1: RGB_VDD -> +5V
- C68 pad 1: RGB_VDD -> +5V
- C69 pad 1: RGB_VDD -> +5V
- C7 pad 1: RGB_VDD -> +5V
- C70 pad 1: RGB_VDD -> +5V
- C71 pad 1: RGB_VDD -> +5V
- C72 pad 1: RGB_VDD -> +5V
- C73 pad 1: RGB_VDD -> +5V
- C74 pad 1: RGB_VDD -> +5V
- C75 pad 1: RGB_VDD -> +5V
- C76 pad 1: RGB_VDD -> +5V
- C77 pad 1: RGB_VDD -> +5V
- C78 pad 1: RGB_VDD -> +5V
- C79 pad 1: RGB_VDD -> +5V
- C8 pad 1: RGB_VDD -> +5V
- C80 pad 1: RGB_VDD -> +5V
- C81 pad 1: RGB_VDD -> +5V
- C82 pad 1: RGB_VDD -> +5V
- C83 pad 1: RGB_VDD -> +5V
- C84 pad 1: RGB_VDD -> +5V
- C85 pad 1: RGB_VDD -> +5V
- C86 pad 1: RGB_VDD -> +5V
- C87 pad 1: RGB_VDD -> +5V
- C88 pad 1: RGB_VDD -> +5V
- C89 pad 1: RGB_VDD -> +5V
- C9 pad 1: RGB_VDD -> +5V
- C90 pad 1: RGB_VDD -> +5V
- C91 pad 1: RGB_VDD -> +5V
- C92 pad 1: RGB_VDD -> +5V
- C93 pad 1: RGB_VDD -> +5V
- C94 pad 1: RGB_VDD -> +5V
- C95 pad 1: RGB_VDD -> +5V
- C96 pad 1: RGB_VDD -> +5V
- C97 pad 1: RGB_VDD -> +5V
- C98 pad 1: RGB_VDD -> +5V
- C99 pad 1: RGB_VDD -> +5V
- RGB1 pad 1: RGB_VDD -> +5V
- RGB10 pad 1: RGB_VDD -> +5V
- RGB11 pad 1: RGB_VDD -> +5V
- RGB12 pad 1: RGB_VDD -> +5V
- RGB13 pad 1: RGB_VDD -> +5V
- RGB14 pad 1: RGB_VDD -> +5V
- RGB14 pad 3: Net-(RGB14-Pad3) -> GND
- RGB15 pad 1: RGB_VDD -> +5V
- RGB15 pad 3: Net-(RGB14-Pad3) -> GND
- RGB16 pad 1: RGB_VDD -> +5V
- RGB16 pad 3: Net-(RGB14-Pad3) -> GND
- RGB17 pad 1: RGB_VDD -> +5V
- RGB17 pad 3: Net-(RGB14-Pad3) -> GND
- RGB18 pad 1: RGB_VDD -> +5V
- RGB18 pad 3: Net-(RGB14-Pad3) -> GND
- RGB19 pad 1: RGB_VDD -> +5V
- RGB19 pad 3: Net-(RGB14-Pad3) -> GND
- RGB2 pad 1: RGB_VDD -> +5V
- RGB20 pad 1: RGB_VDD -> +5V
- RGB20 pad 3: Net-(RGB14-Pad3) -> GND
- RGB21 pad 1: RGB_VDD -> +5V
- RGB21 pad 3: Net-(RGB14-Pad3) -> GND
- RGB22 pad 1: RGB_VDD -> +5V
- RGB22 pad 3: Net-(RGB14-Pad3) -> GND
- RGB23 pad 1: RGB_VDD -> +5V
- RGB23 pad 3: Net-(RGB14-Pad3) -> GND
- RGB24 pad 1: RGB_VDD -> +5V
- RGB24 pad 3: Net-(RGB14-Pad3) -> GND
- RGB25 pad 1: RGB_VDD -> +5V
- RGB25 pad 3: Net-(RGB14-Pad3) -> GND
- RGB26 pad 1: RGB_VDD -> +5V
- RGB26 pad 3: Net-(RGB14-Pad3) -> GND
- RGB27 pad 1: RGB_VDD -> +5V
- RGB27 pad 3: Net-(RGB14-Pad3) -> GND
- RGB28 pad 1: RGB_VDD -> +5V
- RGB28 pad 3: Net-(RGB14-Pad3) -> GND
- RGB29 pad 1: RGB_VDD -> +5V
- RGB29 pad 3: Net-(RGB14-Pad3) -> GND
- RGB3 pad 1: RGB_VDD -> +5V
- RGB30 pad 1: RGB_VDD -> +5V
- RGB30 pad 3: Net-(RGB14-Pad3) -> GND
- RGB31 pad 1: RGB_VDD -> +5V
- RGB31 pad 3: Net-(RGB14-Pad3) -> GND
- RGB32 pad 1: RGB_VDD -> +5V
- RGB32 pad 3: Net-(RGB14-Pad3) -> GND
- RGB33 pad 1: RGB_VDD -> +5V
- RGB34 pad 1: RGB_VDD -> +5V
- RGB35 pad 1: RGB_VDD -> +5V
- RGB36 pad 1: RGB_VDD -> +5V
- RGB37 pad 1: RGB_VDD -> +5V
- RGB38 pad 1: RGB_VDD -> +5V
- RGB39 pad 1: RGB_VDD -> +5V
- RGB4 pad 1: RGB_VDD -> +5V
- RGB40 pad 1: RGB_VDD -> +5V
- RGB41 pad 1: RGB_VDD -> +5V
- RGB42 pad 1: RGB_VDD -> +5V
- RGB43 pad 1: RGB_VDD -> +5V
- RGB44 pad 1: RGB_VDD -> +5V
- RGB45 pad 1: RGB_VDD -> +5V
- RGB46 pad 1: RGB_VDD -> +5V
- RGB47 pad 1: RGB_VDD -> +5V
- RGB48 pad 1: RGB_VDD -> +5V
- RGB49 pad 1: RGB_VDD -> +5V
- RGB5 pad 1: RGB_VDD -> +5V
- RGB50 pad 1: RGB_VDD -> +5V
- RGB51 pad 1: RGB_VDD -> +5V
- RGB52 pad 1: RGB_VDD -> +5V
- RGB53 pad 1: RGB_VDD -> +5V
- RGB54 pad 1: RGB_VDD -> +5V
- RGB55 pad 1: RGB_VDD -> +5V
- RGB56 pad 1: RGB_VDD -> +5V
- RGB57 pad 1: RGB_VDD -> +5V
- RGB58 pad 1: RGB_VDD -> +5V
- RGB59 pad 1: RGB_VDD -> +5V
- RGB6 pad 1: RGB_VDD -> +5V
- RGB60 pad 1: RGB_VDD -> +5V
- RGB61 pad 1: RGB_VDD -> +5V
- RGB62 pad 1: RGB_VDD -> +5V
- RGB63 pad 1: RGB_VDD -> +5V
- RGB64 pad 1: RGB_VDD -> +5V
- RGB65 pad 1: RGB_VDD -> +5V
- RGB66 pad 1: RGB_VDD -> +5V
- RGB67 pad 1: RGB_VDD -> +5V
- RGB68 pad 1: RGB_VDD -> +5V
- RGB69 pad 1: Net-(RGB86-Pad1) -> +5V
- RGB7 pad 1: RGB_VDD -> +5V
- RGB70 pad 1: Net-(RGB86-Pad1) -> +5V
- RGB71 pad 1: Net-(RGB86-Pad1) -> +5V
- RGB72 pad 1: Net-(RGB86-Pad1) -> +5V
- RGB73 pad 1: Net-(RGB86-Pad1) -> +5V
- RGB74 pad 1: Net-(RGB86-Pad1) -> +5V
- RGB75 pad 1: Net-(RGB86-Pad1) -> +5V
- RGB76 pad 1: Net-(RGB86-Pad1) -> +5V
- RGB77 pad 1: Net-(RGB86-Pad1) -> +5V
- RGB78 pad 1: Net-(RGB86-Pad1) -> +5V
- RGB79 pad 1: Net-(RGB86-Pad1) -> +5V
- RGB8 pad 1: RGB_VDD -> +5V
- RGB80 pad 1: Net-(RGB86-Pad1) -> +5V
- RGB81 pad 1: Net-(RGB86-Pad1) -> +5V
- RGB82 pad 1: Net-(RGB86-Pad1) -> +5V
- RGB83 pad 1: Net-(RGB86-Pad1) -> +5V
- RGB84 pad 1: Net-(RGB86-Pad1) -> +5V
- RGB85 pad 1: Net-(RGB86-Pad1) -> +5V
- RGB86 pad 1: Net-(RGB86-Pad1) -> +5V
- RGB87 pad 1: RGB_VDD -> +5V
- RGB88 pad 1: RGB_VDD -> +5V
- RGB89 pad 1: RGB_VDD -> +5V
- RGB9 pad 1: RGB_VDD -> +5V
- RGB90 pad 1: RGB_VDD -> +5V
- RGB91 pad 1: RGB_VDD -> +5V
- RGB92 pad 1: RGB_VDD -> +5V
- RGB93 pad 1: RGB_VDD -> +5V
- RGB94 pad 1: RGB_VDD -> +5V
- RGB95 pad 1: RGB_VDD -> +5V
- RGB96 pad 1: RGB_VDD -> +5V
- RGB97 pad 1: RGB_VDD -> +5V
- RGB98 pad 1: RGB_VDD -> +5V
- RGB99 pad 1: RGB_VDD -> +5V
- TP2 pad 1: RGB_VDD -> 3V3REF
- U1 pad 25: unconnected-(U1-Pad25) -> VBAT
- U1 pad 26: unconnected-(U1-Pad26) -> 3.3V
- U1 pad 27: unconnected-(U1-Pad27) -> GND
- U1 pad 28: unconnected-(U1-Pad28) -> PROGRAM
- U1 pad 29: unconnected-(U1-Pad29) -> RESET
- U1 pad 37: unconnected-(U1-Pad37) -> A21_DAC0
- U1 pad 38: unconnected-(U1-Pad38) -> A22_DAC1
- U1 pad 40: unconnected-(U1-Pad40) -> PIN_13_LED
- U1 pad 41: unconnected-(U1-Pad41) -> PIN_14_A0_SCK0
- U1 pad 42: unconnected-(U1-Pad42) -> PIN_15_A1_CS0
- U1 pad 43: unconnected-(U1-Pad43) -> PIN_16_A2_SCL0
- U1 pad 44: unconnected-(U1-Pad44) -> PIN_17_A3_SDA0
- U1 pad 45: unconnected-(U1-Pad45) -> PIN18_A4_SDA0
- U1 pad 46: unconnected-(U1-Pad46) -> PIN_19_A5_SCL0
- U1 pad 47: unconnected-(U1-Pad47) -> PIN_20_A6
- U1 pad 48: unconnected-(U1-Pad48) -> PIN_21_A7
- U1 pad 49: unconnected-(U1-Pad49) -> PIN_22_A8
- U1 pad 50: unconnected-(U1-Pad50) -> PIN_23_A9
- U1 pad 52: unconnected-(U1-Pad52) -> AGND
- U1 pad 54: VUSB -> +5V
- U1 pad 55: unconnected-(U1-Pad55) -> AREF
- U1 pad 59: unconnected-(U1-Pad59) -> USB_D-
- U1 pad 60: unconnected-(U1-Pad60) -> USB_D+
- U1 pad 61: unconnected-(U1-Pad61) -> GND
- U1 pad 62: unconnected-(U1-Pad62) -> GND
- U2 pad 1: VUSB -> +5V
Other:
- board size 407.7 x 139.9 mm -> 407.7 x 142.5 mm
